Commit message: adding a laser sensor

File: src/articubot_one/description/robot.urdf.xacro (robot description, xacro)
@@ -3,3 +3,4 @@
     <xacro:include filename="robot_core.xacro" />
     <xacro:include filename="gazebo_control.xacro"/>
+    <xacro:include filename="lidar.xacro"/>
 </robot>

File: src/articubot_one/description/robot_core.xacro (robot description, xacro)
@@ -22,4 +22,6 @@
     <xacro:property name="wheel_mass" value="0.1"/>
     <xacro:property name="caster_wheel_mass" value="0.1"/>
+    <xacro:property name="lidar_radius" value="0.03"/>
+    <xacro:property name="lidar_length" value="0.03"/>
     <link name="base_link">
     </link>

Commit message: Solved problem

File: src/articubot_one/description/robot.urdf.xacro (robot description, xacro)
@@ -9,8 +9,5 @@
     </xacro:unless>
     <xacro:include filename="robot_core.xacro" />
-    <!-- <xacro:include filename="gazebo_control.xacro"/> -->
-    <!-- <xacro:include filename="ros2_control.xacro"/>  -->
     <xacro:include filename="lidar.xacro"/>
     <xacro:include filename="camera.xacro"/>
-    <!-- <xacro:include filename="depth_camera.xacro"/> -->
 </robot>

File: src/articubot_one/description/robot_core.xacro (robot description, xacro)
@@ -21,5 +21,5 @@
     <xacro:property name="wheel_radius" value="0.05"/>
     <xacro:property name="wheel_length" value="0.03"/>
-    <xacro:property name="caster_wheel_radius" value="0.02"/>
+    <xacro:property name="caster_wheel_radius" value="0.025"/>
     <xacro:property name="box_mass" value="0.5"/>
     <xacro:property name="wheel_mass" value="0.1"/>
@@ -40,5 +40,5 @@
             <origin xyz="0 0 0"/>
             <geometry>
-                <box size="${box_x} ${box_y} ${box_z}"/>
+                <box size="${box_x-0.001} ${box_y-0.001} ${box_z-0.001}"/>
             </geometry>
         </collision>
@@ -75,5 +75,5 @@
             <origin xyz="0 0 0" rpy="${pi/2} 0 0"/>
             <geometry>
-                <cylinder radius="${wheel_radius}" length="${wheel_length}" />
+                <cylinder radius="${wheel_radius}" length="${wheel_length-0.001}" />
             </geometry>
         </collision>
@@ -104,5 +104,5 @@
             <origin xyz="0 0 0" rpy="${pi/2} 0 0"/>
             <geometry>
-                <cylinder radius="${wheel_radius}" length="${wheel_length}" />
+                <cylinder radius="${wheel_radius}" length="${wheel_length-0.001}" />
             </geometry>
             <material name='blue'/>

Commit message: Add sim_mode toggle for ros2_control

File: src/articubot_one/description/robot.urdf.xacro (robot description, xacro)
@@ -2,4 +2,5 @@
 <robot xmlns:xacro="http://www.ros.org/wiki/xacro" name="bot">
     <xacro:arg name="use_ros2_control" default="true"/>
+    <xacro:arg name="sim_mode" default="true"/>
     <xacro:if value="$(arg use_ros2_control)">
         <xacro:include filename="ros2_control.xacro"/>

File: src/articubot_one/description/ros2_control.xacro (robot description, xacro)
@@ -1,28 +1,61 @@
 <?xml version="1.0"?>
 <robot xmlns:xacro="http://www.ros.org/wiki/xacro">
-    <ros2_control name="GazeboSystem" type="system">
-        <hardware>
-        <plugin>gz_ros2_control/GazeboSimSystem</plugin>
-        </hardware>
-        <joint name="left_wheel_joint">
-            <command_interface name="velocity">
-                <param name="min">-10.0</param>
-                <param name="max">10.0</param>
-            </command_interface>
-            <state_interface name="velocity"/>
-            <state_interface name="position"/>
-        </joint>
-        <joint name="right_wheel_joint">
-            <command_interface name="velocity">
-                <param name="min">-10.0</param>
-                <param name="max">10.0</param>
-            </command_interface>
-            <state_interface name="velocity"/>
-            <state_interface name="position"/>
-        </joint>
-    </ros2_control>
+    <xacro:unless value="$(arg sim_mode)">
+        <ros2_control name="RealRobot" type="systel">
+            <hardware>
+                <plugin>diffdrive_arduino/DiffDriveArduino</plugin>
+                <param name="left_wheel_name">left_wheel_joint</param>
+                <param name="right_wheel_name">right_wheel_joint</param>
+                <param name="loop_rate">30</param>
+                <param name="device">/dev/ttyUSB0</param>
+                <param name="baud_rate">57600</param>
+                <param name="timeout">1000</param>
+                <param name="enc_counts_per_rev">3450</param>
+            </hardware>
+            <joint name="left_wheel_joint">
+                <command_interface name="velocity">
+                    <param name="min">-10.0</param>
+                    <param name="max">10.0</param>
+                </command_interface>
+                <state_interface name="velocity"/>
+                <state_interface name="position"/>
+            </joint>
+            <joint name="right_wheel_joint">
+                <command_interface name="velocity">
+                    <param name="min">-10.0</param>
+                    <param name="max">10.0</param>
+                </command_interface>
+                <state_interface name="velocity"/>
+                <state_interface name="position"/>
+            </joint>
+        </ros2_control>
+    </xacro:unless>
+    <xacro:if value="$(arg sim_mode)">
+        <ros2_control name="GazeboSystem" type="system">
+            <hardware>
+            <plugin>gz_ros2_control/GazeboSimSystem</plugin>
+            </hardware>
+            <joint name="left_wheel_joint">
+                <command_interface name="velocity">
+                    <param name="min">-10.0</param>
+                    <param name="max">10.0</param>
+                </command_interface>
+                <state_interface name="velocity"/>
+                <state_interface name="position"/>
+            </joint>
+            <joint name="right_wheel_joint">
+                <command_interface name="velocity">
+                    <param name="min">-10.0</param>
+                    <param name="max">10.0</param>
+                </command_interface>
+                <state_interface name="velocity"/>
+                <state_interface name="position"/>
+            </joint>
+        </ros2_control>
+    </xacro:if>
     <gazebo>
         <plugin name="gz_ros2_control::GazeboSimROS2ControlPlugin" filename="libgz_ros2_control-system.so">
             <parameters>$(find articubot_one)/config/my_controllers.yaml</parameters>
+            <parameters>$(find articubot_one)/config/gz_ros2_ctl_use_sim.yaml</parameters>
         </plugin>
     </gazebo>
