Commit message: Changes added, shocks in the bot presists

File: src/articubot_one/description/robot_core.xacro (robot description, xacro)
@@ -21,8 +21,8 @@
     <xacro:property name="wheel_radius" value="0.05"/>
     <xacro:property name="wheel_length" value="0.03"/>
-    <xacro:property name="caster_wheel_radius" value="0.025"/>
+    <xacro:property name="caster_wheel_radius" value="0.02"/>
     <xacro:property name="box_mass" value="0.5"/>
     <xacro:property name="wheel_mass" value="0.1"/>
-    <xacro:property name="caster_wheel_mass" value="0.1"/>
+    <xacro:property name="caster_wheel_mass" value="1"/>
     <xacro:property name="lidar_radius" value="0.03"/>
     <xacro:property name="lidar_length" value="0.03"/>
@@ -157,5 +157,5 @@
         </inertial>
     </link>
-    <gazebo reference="caster_wheel">
+    <!-- <gazebo reference="caster_wheel">
         <visual>
             <material>
@@ -167,4 +167,16 @@
         <mu1 value="0.001"/>
         <mu2 value="0.001"/>
+    </gazebo> -->
+    <gazebo reference="caster_wheel">
+        <mu1 value="0.001"/>
+        <mu2 value="0.001"/>
+        <surface>
+        <friction>
+            <ode>
+            <mu>0.001</mu>
+            <mu2>0.001</mu2>
+            </ode>
+        </friction>
+        </surface>
     </gazebo>
     <joint name="caster_wheel_joint" type="fixed">

Commit message: Shockes solved

File: src/articubot_one/description/robot_core.xacro (robot description, xacro)
@@ -24,5 +24,5 @@
     <xacro:property name="box_mass" value="0.5"/>
     <xacro:property name="wheel_mass" value="0.1"/>
-    <xacro:property name="caster_wheel_mass" value="1"/>
+    <xacro:property name="caster_wheel_mass" value="0.05"/>
     <xacro:property name="lidar_radius" value="0.03"/>
     <xacro:property name="lidar_length" value="0.03"/>

Commit message: Working well

File: src/articubot_one/description/robot_core.xacro (robot description, xacro)
@@ -97,5 +97,5 @@
         <parent link="base_link"/>
         <child link="left_wheel"/>
-        <origin xyz="${-box_x/2+wheel_radius} ${box_y/2+wheel_length/2} ${wheel_radius}" rpy="0 0 0"/>
+        <origin xyz="${-box_x/2+wheel_radius} ${box_y/2+wheel_length/2+0.01} ${wheel_radius}" rpy="0 0 0"/>
         <axis xyz="0 1 0" />
     </joint>
@@ -133,5 +133,5 @@
         <parent link="base_link"/>
         <child link="right_wheel"/>
-        <origin xyz="${-box_x/2+wheel_radius} ${-box_y/2-wheel_length/2} ${wheel_radius}" rpy="0 0 0"/>
+        <origin xyz="${-box_x/2+wheel_radius} ${-box_y/2-wheel_length/2-0.01} ${wheel_radius}" rpy="0 0 0"/>
         <axis xyz="0 1 0" />
     </joint>
@@ -139,5 +139,5 @@
         <visual>
             <geometry>
-                <sphere radius="${caster_wheel_radius}" />
+                <sphere radius="${caster_wheel_radius-0.001}" />
             </geometry>
             <origin xyz="0 0 ${-caster_wheel_radius}" />

Commit message: Add slam_toolbox and map topic

File: src/articubot_one/description/robot_core.xacro (robot description, xacro)
@@ -29,4 +29,11 @@
     <link name="base_link">
     </link>
+    <link name="base_footprint">
+    </link>
+    <joint name="base_footprint_joint" type="fixed">
+        <parent link="base_link" />
+        <child link="base_footprint" />
+        <origin xyz="0 0 0" rpy="0 0 0" />
+    </joint>
     <link name="chassis">
         <visual>
