Commit message: Added lidar and followed convection

File: src/articubot_one/description/lidar.xacro (robot description, xacro)
@@ -3,8 +3,8 @@
     <joint name="lidar_joint" type="fixed">
         <parent link="chassis"/>
-        <child link="lidar_link"/>
+            <child link="laser_frame"/>
         <origin xyz="0 0 0.045" rpy="0 0 0"/>
     </joint>
-    <link name="lidar_link">
+    <link name="laser_frame">
         <visual>
             <geometry>
@@ -18,4 +18,11 @@
             </geometry>
         </collision>
+        <inertial>
+            <mass value="0.1" />
+            <origin xyz="0 0 0" rpy="0 0 0"/>
+            <inertia ixx="0.0001" ixy="0.0" ixz="0.0"
+                     iyy="0.0001" iyz="0.0"
+                     izz="0.0001" />
+        </inertial>
     </link>
     <gazebo reference="laser_frame">

Commit message: hello

File: src/articubot_one/description/lidar.xacro (robot description, xacro)
@@ -48,5 +48,5 @@
         </lidar>
         <plugin filename="gz-sim-sensors-system" name="gz::sim::systems::Sensors">
-            <render_engine>ogre2</render_engine>
+            <render_engine>ogre</render_engine>
         </plugin>
     </sensor>

File: src/articubot_one/description/robot.urdf.xacro (robot description, xacro)
@@ -4,3 +4,4 @@
     <xacro:include filename="gazebo_control.xacro"/>
     <xacro:include filename="lidar.xacro"/>
+    <!-- <xacro:include filename="camera.xacro"/> -->
 </robot>

File: src/articubot_one/description/robot_core.xacro (robot description, xacro)
@@ -12,4 +12,7 @@
     <material name="black">
         <color rgba="0 0 0 1" />
+    </material>
+    <material name="pink">
+        <color rgba="0.7 0.09 0.5 1" />
     </material>
     <xacro:property name="box_x" value="0.3"/>

Commit message: Synchronization issue debugged

File: src/articubot_one/description/lidar.xacro (robot description, xacro)
@@ -3,5 +3,5 @@
     <joint name="lidar_joint" type="fixed">
         <parent link="chassis"/>
-            <child link="laser_frame"/>
+        <child link="laser_frame"/>
         <origin xyz="0 0 0.045" rpy="0 0 0"/>
     </joint>
@@ -30,5 +30,5 @@
         <visualize>true</visualize>
         <always_on>true</always_on>
-        <update_rate>10</update_rate>
+        <update_rate>30</update_rate>
         <topic>scan</topic> <gz_frame_id>laser_frame</gz_frame_id>
         <lidar>

Commit message: Working on robotic arm

File: src/articubot_one/description/lidar.xacro (robot description, xacro)
@@ -4,5 +4,5 @@
         <parent link="chassis"/>
         <child link="laser_frame"/>
-        <origin xyz="0 0 0.045" rpy="0 0 0"/>
+        <origin xyz="${box_x/2-lidar_radius} 0 0.045" rpy="0 0 0"/>
     </joint>
     <link name="laser_frame">

File: src/articubot_one/description/robot.urdf.xacro (robot description, xacro)
@@ -12,3 +12,5 @@
     <xacro:include filename="lidar.xacro"/>
     <xacro:include filename="camera.xacro"/>
+    <xacro:include filename="imu.xacro"/>
+    <xacro:include filename="robotic_arm.xacro"/>
 </robot>
